File: kolyscon_Board.kicad_sch (KiCad schematic)
At the start: 41 parts, among them Q1 CJ2310, Q10 CJ2310, Q11 CJ2310, Q2 CJ2310, Q3 CJ2310, Q4 CJ2310, Q5 CJ2310, Q6 CJ2310, Q7 CJ2310, Q8 CJ2310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

Commit message: Schematics changes
Parts:
- added D1: D, symbol Device:D
- added U3: ~, symbol kolyscon_Symbols:Weird_Purple_RP2040_Board
- ENC1, ENC2: footprint (none) -> Connector_JST:JST_XH_B4B-XH-A_1x04_P2.50mm_Vertical
- Q1, Q10, Q11, Q2, Q3, Q4, Q5, Q6, Q7, Q8, Q9: value CJ2310 -> HL2302
- R1, R10, R11, R2, R3, R4, R5, R6, R7, R8, R9: footprint (none) -> Resistor_SMD:R_0603_1608Metric
- WLED1, WLED2, WLED3, WLED4: footprint (none) -> Connector_JST:JST_XH_B3B-XH-A_1x03_P2.50mm_Vertical
Connections:
- net +5V: now also D1.1 (K)
- new net: D1.2 (A), U3.44 (VBUS)
Other:
- moved on the sheet: WLED3, WLED4

Commit message: Some schema work
Parts:
- removed D1: D, symbol Device:D
- added J1: Conn_01x04, kolyscon_Board_Footprints:USB-C_Conn_Small, symbol Connector_Generic:Conn_01x04
- U3: footprint (none) -> kolyscon_Board_Footprints:WeirdPurpleRP2040Board
Connections:
- net +5V: now also ENC1.4 (Pin_4), ENC2.4 (Pin_4), U3.44 (VBUS); no longer ENC1.3 (Pin_3), ENC2.3 (Pin_3), WLED1.1 (Pin_1), WLED2.1 (Pin_1), WLED3.1 (Pin_1), WLED4.1 (Pin_1)
- net BT_D_1: now also U3.4 (3); no longer B10.1 (Pin_1), B11.1 (Pin_1), B2.1 (Pin_1), B3.1 (Pin_1), B4.1 (Pin_1), B5.1 (Pin_1), B6.1 (Pin_1), B7.1 (Pin_1), B8.1 (Pin_1), B9.1 (Pin_1)
- net ENC_1_A: now also U3.29 (22)
- net ENC_1_B: now also U3.30 (23)
- net ENC_2_A: now also U3.31 (24)
- net ENC_2_B: now also U3.32 (25)
- net GND: now also ENC1.3 (Pin_3), ENC2.3 (Pin_3), U3.39 (GND), U3.42 (GND), WLED1.1 (Pin_1), WLED2.1 (Pin_1), WLED3.1 (Pin_1), WLED4.1 (Pin_1), J1.1 (Pin_1); no longer ENC1.4 (Pin_4), ENC2.4 (Pin_4), WLED1.3 (Pin_3), WLED2.3 (Pin_3), WLED3.3 (Pin_3), WLED4.3 (Pin_3)
- net SHIFTREG_CLK: now also U3.2 (1)
- net SHIFTREG_LATCH: now also U3.3 (2)
- net SHIFTREG_SER: now also U3.1 (0)
- net WLED_1: now also U3.25 (18)
- net WLED_2: now also U3.26 (19)
- net WLED_3: now also U3.27 (20)
- net WLED_4: now also U3.28 (21)
- net BT_D_6: now reaches U3.10 (8)
- net BT_D_6: now also B6.1 (Pin_1)
- net BT_D_7: now reaches U3.11 (9)
- net BT_D_7: now also B7.1 (Pin_1)
- net BT_D_8: now reaches U3.12 (10)
- net BT_D_8: now also B8.1 (Pin_1)
- net BT_D_9: now reaches U3.13 (11)
- net BT_D_9: now also B9.1 (Pin_1)
- net BT_D_10: now reaches U3.14 (12)
- net BT_D_10: now also B10.1 (Pin_1)
- net BT_D_11: now reaches U3.16 (13)
- net BT_D_11: now also B11.1 (Pin_1)
- net BT_D_2: now reaches U3.5 (4)
- net BT_D_2: now also B2.1 (Pin_1)
- net BT_D_4: now reaches U3.7 (6)
- net BT_D_4: now also B4.1 (Pin_1)
- net BT_D_3: now reaches U3.8 (5)
- net BT_D_3: now also B3.1 (Pin_1)
- net BT_D_5: now reaches U3.9 (7)
- net BT_D_5: now also B5.1 (Pin_1)
- new net +5V_PWR: J1.4 (Pin_4), WLED1.3 (Pin_3), WLED2.3 (Pin_3), WLED3.3 (Pin_3), WLED4.3 (Pin_3)
- no-connect marks 6 -> 27

Commit message: Schema work
Parts:
- added H1, H2, H3, H4: MountingHole, MountingHole:MountingHole_3.2mm_M3, symbol Mechanical:MountingHole
Connections:
- net GND: no longer J1.1 (Pin_1), WLED1.1 (Pin_1), WLED2.1 (Pin_1), WLED3.1 (Pin_1), WLED4.1 (Pin_1)
- new net GND_PWR: J1.1 (Pin_1), WLED1.1 (Pin_1), WLED2.1 (Pin_1), WLED3.1 (Pin_1), WLED4.1 (Pin_1)
Other:
- moved on the sheet: WLED1, WLED2, WLED3, WLED4

Commit message: -Routing
Parts:
- ENC1, ENC2, J1, U1, U2, U3, WLED1, WLED2, WLED3, WLED4: now left out of the parts list
- Q1, Q10, Q11, Q2, Q3, Q4, Q5, Q6, Q8, Q9: value HL2302 -> ~; LCSC (none) -> C28646271
- Q7: value HL2302 -> ~
- R1, R10, R11, R2, R3, R4, R5, R6, R7, R8, R9: value R -> R1k; LCSC (none) -> C21190
Connections:
- net GND_PWR is gone; now on net GND: J1.1 (Pin_1), WLED1.1 (Pin_1), WLED2.1 (Pin_1), WLED3.1 (Pin_1), WLED4.1 (Pin_1)
- net BT_D_1: now also U3.9 (7); no longer U3.4 (3)
- net BT_D_10: now also U3.27 (20); no longer U3.14 (12)
- net BT_D_11: now also U3.28 (21); no longer U3.16 (13)
- net BT_D_2: now also U3.10 (8); no longer U3.5 (4)
- net BT_D_3: now also U3.11 (9); no longer U3.8 (5)
- net BT_D_4: now also U3.12 (10); no longer U3.7 (6)
- net BT_D_5: now also U3.16 (13); no longer U3.9 (7)
- net BT_D_6: now also U3.14 (12); no longer U3.10 (8)
- net BT_D_7: now also U3.13 (11); no longer U3.11 (9)
- net BT_D_8: now also U3.25 (18); no longer U3.12 (10)
- net BT_D_9: now also U3.26 (19); no longer U3.13 (11)
- net ENC_1_A: now also U3.4 (3); no longer U3.29 (22)
- net ENC_1_B: now also U3.5 (4); no longer U3.30 (23)
- net ENC_2_A: now also U3.7 (5); no longer U3.31 (24)
- net ENC_2_B: now also U3.8 (6); no longer U3.32 (25)
- net GND: now also U3.15 (GND), U3.6 (GND)
- net WLED_1: now also U3.29 (22); no longer U3.25 (18)
- net WLED_2: now also U3.30 (23); no longer U3.26 (19)
- net WLED_3: now also U3.31 (24); no longer U3.27 (20)
- net WLED_4: now also U3.32 (25); no longer U3.28 (21)
- no-connect marks 27 -> 25
Other:
- moved on the sheet: U3

Commit message: Some refactors and fixes
Parts:
- B1, B10, B11, B2, B3, B4, B5, B6, B7, B8, B9: now left out of the parts list
- Q1, Q10, Q11, Q2, Q3, Q4, Q5, Q6, Q8, Q9: footprint Package_TO_SOT_SMD:SOT-23 -> Package_TO_SOT_SMD:SOT-23-3; LCSC C28646271 -> (none)
- Q7: footprint Package_TO_SOT_SMD:SOT-23 -> Package_TO_SOT_SMD:SOT-23-3
- R1, R10, R11, R2, R3, R4, R5, R6, R7, R8, R9: value R1k -> R2k; LCSC C21190 -> (none)
Connections:
- net +5V: no longer U1.10 (~{SRCLR}), U1.16 (VCC), U2.10 (~{SRCLR}), U2.16 (VCC)
- net +3.3V: now reaches U3.40 (3V3)
- net +3.3V: now also U1.10 (~{SRCLR}), U1.16 (VCC), U2.10 (~{SRCLR}), U2.16 (VCC)
- no-connect marks 25 -> 24

Commit message: Board refactors and fixes
Parts:
- Q1, Q10, Q11, Q2, Q3, Q4, Q5, Q6, Q7, Q8, Q9: footprint Package_TO_SOT_SMD:SOT-23-3 -> Package_TO_SOT_THT:TO-92_Inline; symbol Device:Q_NMOS_GSD -> Transistor_BJT:Q_NPN_CBE
- R1, R10, R11, R2, R3, R4, R5, R6, R7, R8, R9: footprint Resistor_SMD:R_0603_1608Metric -> Resistor_THT:R_Axial_DIN0204_L3.6mm_D1.6mm_P1.90mm_Vertical
Connections:
- net GND: now also Q1.3 (E), Q10.3 (E), Q11.3 (E), Q2.3 (E), Q3.3 (E), Q4.3 (E), Q5.3 (E), Q6.3 (E), Q7.3 (E), Q8.3 (E), Q9.3 (E); no longer Q1.2 (S), Q10.2 (S), Q11.2 (S), Q2.2 (S), Q3.2 (S), Q4.2 (S), Q5.2 (S), Q6.2 (S), Q7.2 (S), Q8.2 (S), Q9.2 (S)
- net at R6.1: now also Q6.2 (B); no longer Q6.1 (G)
- net at R1.1: now also Q1.2 (B); no longer Q1.1 (G)
- net at Q4.1 (C): now also B4.2 (Pin_2); no longer R4.1
- net at Q11.1 (C): now also B11.2 (Pin_2); no longer R11.1
- net at B6.2 (Pin_2): now also Q6.1 (C); no longer Q6.3 (D)
- net at B5.2 (Pin_2): now also Q5.1 (C); no longer Q5.3 (D)
- net at R2.1: now also Q2.2 (B); no longer Q2.1 (G)
- net at B2.2 (Pin_2): now also Q2.1 (C); no longer Q2.3 (D)
- net at B10.2 (Pin_2): now also Q10.1 (C); no longer Q10.3 (D)
- net at R10.1: now also Q10.2 (B); no longer Q10.1 (G)
- net at R5.1: now also Q5.2 (B); no longer Q5.1 (G)
- net at Q9.1 (C): now also B9.2 (Pin_2); no longer R9.1
- net at Q8.1 (C): now also B8.2 (Pin_2); no longer R8.1
- net at B7.2 (Pin_2): now also Q7.1 (C); no longer Q7.3 (D)
- net at B1.2 (Pin_2): now also Q1.1 (C); no longer Q1.3 (D)
- net at Q3.1 (C): now also B3.2 (Pin_2); no longer R3.1
- net at R7.1: now also Q7.2 (B); no longer Q7.1 (G)
- new net: Q4.2 (B), R4.1
- new net: Q11.2 (B), R11.1
- new net: Q9.2 (B), R9.1
- new net: Q8.2 (B), R8.1
- new net: Q3.2 (B), R3.1
Changed lines of the file:
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@@
 (kicad_sch
-	(version 20231120)
+	(version 20250114)
 	(generator "eeschema")
-	(generator_version "8.0")
+	(generator_version "9.0")
 	(paper "A4")
 	(junction
@@
 			)
 		)
-		(property "Footprint" "Resistor_SMD:R_0603_1608Metric"
+		(property "Footprint" "Resistor_THT:R_Axial_DIN0204_L3.6mm_D1.6mm_P1.90mm_Vertical"
 			(at 279.908 24.13 90)
 			(effects
@@
 			)
 		)
-		(property "Footprint" "Resistor_SMD:R_0603_1608Metric"
+		(property "Footprint" "Resistor_THT:R_Axial_DIN0204_L3.6mm_D1.6mm_P1.90mm_Vertical"
 			(at 156.718 24.13 90)
 			(effects
@@
 	)
 	(symbol
-		(lib_id "Device:Q_NMOS_GSD")
+		(lib_id "Transistor_BJT:Q_NPN_CBE")
 		(at 222.25 27.94 180)
 		(unit 1)
@@
 			)
 		)
-		(property "Footprint" "Package_TO_SOT_SMD:SOT-23-3"
+		(property "Footprint" "Package_TO_SOT_THT:TO-92_Inline"
 			(at 217.17 30.48 0)
 			(effects
@@
 			)
 		)
-		(property "Description" "N-MOSFET transistor, gate/source/drain"
+		(property "Description" "NPN transistor, collector/base/emitter"
 			(at 222.25 27.94 0)
 			(effects
@@
 	)
 	(symbol
-		(lib_id "Device:Q_NMOS_GSD")
+		(lib_id "Transistor_BJT:Q_NPN_CBE")
 		(at 273.05 66.04 180)
 		(unit 1)
@@
 			)
 		)
-		(property "Footprint" "Package_TO_SOT_SMD:SOT-23-3"
+		(property "Footprint" "Package_TO_SOT_THT:TO-92_Inline"
 			(at 267.97 68.58 0)
 			(effects
@@
 			)
 		)
-		(property "Description" "N-MOSFET transistor, gate/source/drain"
+		(property "Description" "NPN transistor, collector/base/emitter"
 			(at 273.05 66.04 0)
 			(effects
@@
 	)
 	(symbol
-		(lib_id "Device:Q_NMOS_GSD")
+		(lib_id "Transistor_BJT:Q_NPN_CBE")
 		(at 273.05 27.94 180)
 		(unit 1)
@@
 			)
 		)
-		(property "Footprint" "Package_TO_SOT_SMD:SOT-23-3"
+		(property "Footprint" "Package_TO_SOT_THT:TO-92_Inline"
 			(at 267.97 30.48 0)
 			(effects
@@
 			)
 		)
-		(property "Description" "N-MOSFET transistor, gate/source/drain"
+		(property "Description" "NPN transistor, collector/base/emitter"
 			(at 273.05 27.94 0)
 			(effects
@@
 			)
 		)
-		(property "Footprint" "Resistor_SMD:R_0603_1608Metric"
+		(property "Footprint" "Resistor_THT:R_Axial_DIN0204_L3.6mm_D1.6mm_P1.90mm_Vertical"
 			(at 279.908 62.23 90)
 			(effects
@@
 			)
 		)
-		(property "Footprint" "Resistor_SMD:R_0603_1608Metric"
+		(property "Footprint" "Resistor_THT:R_Axial_DIN0204_L3.6mm_D1.6mm_P1.90mm_Vertical"
 			(at 179.578 24.13 90)
 			(effects
@@
 	)
 	(symbol
-		(lib_id "Device:Q_NMOS_GSD")
+		(lib_id "Transistor_BJT:Q_NPN_CBE")
 		(at 245.11 66.04 180)
 		(unit 1)
@@
 			)
 		)
-		(property "Footprint" "Package_TO_SOT_SMD:SOT-23-3"
+		(property "Footprint" "Package_TO_SOT_THT:TO-92_Inline"
 			(at 240.03 68.58 0)
 			(effects
@@
 			)
 		)
-		(property "Description" "N-MOSFET transistor, gate/source/drain"
+		(property "Description" "NPN transistor, collector/base/emitter"
 			(at 245.11 66.04 0)
 			(effects
@@
 			)
 		)
-		(property "Footprint" "Resistor_SMD:R_0603_1608Metric"
+		(property "Footprint" "Resistor_THT:R_Axial_DIN0204_L3.6mm_D1.6mm_P1.90mm_Vertical"
 			(at 254.508 24.13 90)
 			(effects
@@
 	)
 	(symbol
-		(lib_id "Device:Q_NMOS_GSD")
+		(lib_id "Transistor_BJT:Q_NPN_CBE")
 		(at 247.65 27.94 180)
 		(unit 1)
@@
 			)
 		)
-		(property "Footprint" "Package_TO_SOT_SMD:SOT-23-3"
+		(property "Footprint" "Package_TO_SOT_THT:TO-92_Inline"
 			(at 242.57 30.48 0)
 			(effects
@@
 			)
 		)
-		(property "Description" "N-MOSFET transistor, gate/source/drain"
+		(property "Description" "NPN transistor, collector/base/emitter"
 			(at 247.65 27.94 0)
 			(effects
@@
 	)
 	(symbol
-		(lib_id "Device:Q_NMOS_GSD")
+		(lib_id "Transistor_BJT:Q_NPN_CBE")
 		(at 219.71 66.04 180)
 		(unit 1)
@@
 			)
 		)
-		(property "Footprint" "Package_TO_SOT_SMD:SOT-23-3"
+		(property "Footprint" "Package_TO_SOT_THT:TO-92_Inline"
 			(at 214.63 68.58 0)
 			(effects
@@
 			)
 		)
-		(property "Description" "N-MOSFET transistor, gate/source/drain"
+		(property "Description" "NPN transistor, collector/base/emitter"
 			(at 219.71 66.04 0)
 			(effects
@@
 	)
 	(symbol
-		(lib_id "Device:Q_NMOS_GSD")
+		(lib_id "Transistor_BJT:Q_NPN_CBE")
 		(at 194.31 66.04 180)
 		(unit 1)
@@
 			)
 		)
-		(property "Footprint" "Package_TO_SOT_SMD:SOT-23-3"
+		(property "Footprint" "Package_TO_SOT_THT:TO-92_Inline"
 			(at 189.23 68.58 0)
 			(effects
@@
 			)
 		)
-		(property "Description" "N-MOSFET transistor, gate/source/drain"
+		(property "Description" "NPN transistor, collector/base/emitter"
 			(at 194.31 66.04 0)
 			(effects
@@
 	)
 	(symbol
-		(lib_id "Device:Q_NMOS_GSD")
+		(lib_id "Transistor_BJT:Q_NPN_CBE")
 		(at 172.72 27.94 180)
 		(unit 1)
@@
 			)
 		)
-		(property "Footprint" "Package_TO_SOT_SMD:SOT-23-3"
+		(property "Footprint" "Package_TO_SOT_THT:TO-92_Inline"
 			(at 167.64 30.48 0)
 			(effects
@@
 			)
 		)
-		(property "Description" "N-MOSFET transistor, gate/source/drain"
+		(property "Description" "NPN transistor, collector/base/emitter"
 			(at 172.72 27.94 0)
 			(effects
@@
 	)
 	(symbol
-		(lib_id "Device:Q_NMOS_GSD")
+		(lib_id "Transistor_BJT:Q_NPN_CBE")
 		(at 198.12 27.94 180)
 		(unit 1)
@@
 			)
 		)
-		(property "Footprint" "Package_TO_SOT_SMD:SOT-23-3"
+		(property "Footprint" "Package_TO_SOT_THT:TO-92_Inline"
 			(at 193.04 30.48 0)
 			(effects
@@
 			)
 		)
-		(property "Description" "N-MOSFET transistor, gate/source/drain"
+		(property "Description" "NPN transistor, collector/base/emitter"
 			(at 198.12 27.94 0)
 			(effects
@@
 			)
 		)
-		(property "Footprint" "Resistor_SMD:R_0603_1608Metric"
+		(property "Footprint" "Resistor_THT:R_Axial_DIN0204_L3.6mm_D1.6mm_P1.90mm_Vertical"
 			(at 204.978 24.13 90)
 			(effects
@@
 			)
 		)
-		(property "Footprint" "Resistor_SMD:R_0603_1608Metric"
+		(property "Footprint" "Resistor_THT:R_Axial_DIN0204_L3.6mm_D1.6mm_P1.90mm_Vertical"
 			(at 251.968 62.23 90)
 			(effects
@@
 			)
 		)
-		(property "Footprint" "Resistor_SMD:R_0603_1608Metric"
+		(property "Footprint" "Resistor_THT:R_Axial_DIN0204_L3.6mm_D1.6mm_P1.90mm_Vertical"
 			(at 201.168 62.23 90)
 			(effects
@@
 	)
 	(symbol
-		(lib_id "Device:Q_NMOS_GSD")
+		(lib_id "Transistor_BJT:Q_NPN_CBE")
 		(at 149.86 27.94 180)
 		(unit 1)
@@
 			)
 		)
-		(property "Footprint" "Package_TO_SOT_SMD:SOT-23-3"
+		(property "Footprint" "Package_TO_SOT_THT:TO-92_Inline"
 			(at 144.78 30.48 0)
 			(effects
@@
 			)
 		)
-		(property "Description" "N-MOSFET transistor, gate/source/drain"
+		(property "Description" "NPN transistor, collector/base/emitter"
 			(at 149.86 27.94 0)
 			(effects
@@
 	)
 	(symbol
-		(lib_id "Device:Q_NMOS_GSD")
+		(lib_id "Transistor_BJT:Q_NPN_CBE")
 		(at 168.91 66.04 180)
 		(unit 1)
@@
 			)
 		)
-		(property "Footprint" "Package_TO_SOT_SMD:SOT-23-3"
+		(property "Footprint" "Package_TO_SOT_THT:TO-92_Inline"
 			(at 163.83 68.58 0)
 			(effects
@@
 			)
 		)
-		(property "Description" "N-MOSFET transistor, gate/source/drain"
+		(property "Description" "NPN transistor, collector/base/emitter"
 			(at 168.91 66.04 0)
 			(effects
@@
 			)
 		)
-		(property "Footprint" "Resistor_SMD:R_0603_1608Metric"
+		(property "Footprint" "Resistor_THT:R_Axial_DIN0204_L3.6mm_D1.6mm_P1.90mm_Vertical"
 			(at 226.568 62.23 90)
 			(effects
@@
 			)
 		)
-		(property "Footprint" "Resistor_SMD:R_0603_1608Metric"
+		(property "Footprint" "Resistor_THT:R_Axial_DIN0204_L3.6mm_D1.6mm_P1.90mm_Vertical"
 			(at 175.768 62.23 90)
 			(effects
@@
 			)
 		)
-		(property "Footprint" "Resistor_SMD:R_0603_1608Metric"
+		(property "Footprint" "Resistor_THT:R_Axial_DIN0204_L3.6mm_D1.6mm_P1.90mm_Vertical"
 			(at 229.108 24.13 90)
 			(effects
@@
 		)
 	)
+	(embedded_fonts no)
 )
